Commit message: cleaned up compliance control code with updated urdf with shunk sdh2 hand

File: single_lwr_example/single_lwr_robot/robot/single_lwr_robot_epiaggio.urdf.xacro (robot description, xacro)
@@ -3,8 +3,4 @@
 	<!-- Include all models -->
 	<xacro:include filename="$(find lwr_description)/model/kuka_lwr.urdf.xacro"/>
-	<!-- adapter -->
-  	<xacro:include filename="$(find kuka_lbr4_fkie)/urdf/adapter/adapter.urdf.xacro" />
-  	<!-- sdh -->
-  	<xacro:include filename="$(find kuka_lbr4_fkie)/urdf/sdh/sdh.urdf.xacro" />
 	<!-- and assemble your robot -->
 	<link name="box">
@@ -37,11 +33,3 @@
 		<origin xyz="0 0 1" rpy="0 0 0"/>
 	</xacro:kuka_lwr>
-	<!-- adapter -->
-	<xacro:adapter name="adapter" parent="lwr_7_link">
-		<origin xyz="0 0 0.02" rpy="0 0 0" />
-	</xacro:adapter>
-	<!-- sdh -->
-	<xacro:sdh name="sdh" parent="fws_link">
-		<origin xyz="0 0 0.005" rpy="0 0 0" />
-	</xacro:sdh>
 </robot>
